Commit message: using velodyne_simulator instead of generic gazebo block laser, added launch files + world models

File: urdf/quadrotor_with_velodyne_puck.gazebo.xacro (robot description, xacro)
@@ -1,5 +1,5 @@
 <?xml version="1.0"?>
 <robot name="quadrotor" xmlns:xacro="http://www.ros.org/wiki/xacro">
-    <xacro:include filename="$(find hector_quadrotor_description)/urdf/quadrotor_with_velodyne_puck.urdf.xacro" />
+    <xacro:include filename="$(find joscha_copter)/urdf/quadrotor_with_velodyne_puck.urdf.xacro" />
     <xacro:include filename="$(find hector_quadrotor_gazebo)/urdf/quadrotor_plugins.gazebo.xacro" />
 </robot>

File: urdf/quadrotor_with_velodyne_puck.urdf.xacro (robot description, xacro)
@@ -7,7 +7,7 @@
     <xacro:quadrotor_base_macro />
     <!-- Hokuyo UTM-30LX mounted upside down below the quadrotor body -->
-    <xacro:include filename="$(find hector_quadrotor_description)/urdf/velodyne_puck.xacro" />
-    <xacro:velodyne_puck name="laser0" parent="base_link" ros_topic="scan" update_rate="10" >
-      <origin xyz="0.0 0.0 -0.097" rpy="0 0 0"/>
-    </xacro:velodyne_puck>
+    <xacro:include filename="$(find velodyne_description)/urdf/VLP-16.urdf.xacro"/>
+    <VLP-16 parent="base_link" name="velodyne" topic="/velodyne_points">
+    <origin xyz="0 0 -0.097" rpy="0 0 0" />
+    </VLP-16>
 </robot>
